File: DS3231.kicad_pcb (KiCad board)
At the start: 2 copper layers, 22.9 x 17.8 mm, 9 parts, among them IC1 DS3231, J1 Conn_01x08_Pin

Commit message: fix: use the Keystone 3000 battery holder
Parts:
- B1: footprint external_footprints:CR1220 -> Battery:BatteryHolder_Keystone_3000_1x12mm
- moved B1 0.42 mm to (148.6, 102.8)
Routing:
- net /VBAT: track 23.2 -> 44.9 mm
- net 3.3V: track 25.1 -> 27.1 mm

Commit message: fix: ground DS3231 pins 5 to 12
The datasheet says these N.C. pins must be connected to ground, they
were left open. Rename them GND in the symbol, wire them to GND and
connect the pads in the layout.
Connections:
- IC1 pad 10: unconnected-(IC1-NC5-Pad10) -> GND
- IC1 pad 11: unconnected-(IC1-NC6-Pad11) -> GND
- IC1 pad 12: unconnected-(IC1-NC7-Pad12) -> GND
- IC1 pad 5: unconnected-(IC1-NC-Pad5) -> GND
- IC1 pad 6: unconnected-(IC1-NC1-Pad6) -> GND
- IC1 pad 7: unconnected-(IC1-NC2-Pad7) -> GND
- IC1 pad 8: unconnected-(IC1-NC3-Pad8) -> GND
- IC1 pad 9: unconnected-(IC1-NC4-Pad9) -> GND
Changed lines of the file:
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@@
 			(layers "F.Cu" "F.Mask" "F.Paste")
 			(roundrect_rratio 0.25)
-			(net "unconnected-(IC1-NC-Pad5)")
-			(pinfunction "NC_5")
-			(pintype "passive+no_connect")
+			(net "GND")
+			(pinfunction "GND_5")
+			(pintype "passive")
 		)
 		(pad "6" smd roundrect
@@
 			(layers "F.Cu" "F.Mask" "F.Paste")
 			(roundrect_rratio 0.25)
-			(net "unconnected-(IC1-NC1-Pad6)")
-			(pinfunction "NC1_6")
-			(pintype "passive+no_connect")
+			(net "GND")
+			(pinfunction "GND_6")
+			(pintype "passive")
 		)
 		(pad "7" smd roundrect
@@
 			(layers "F.Cu" "F.Mask" "F.Paste")
 			(roundrect_rratio 0.25)
-			(net "unconnected-(IC1-NC2-Pad7)")
-			(pinfunction "NC2_7")
-			(pintype "passive+no_connect")
+			(net "GND")
+			(pinfunction "GND_7")
+			(pintype "passive")
 		)
 		(pad "8" smd roundrect
@@
 			(layers "F.Cu" "F.Mask" "F.Paste")
 			(roundrect_rratio 0.25)
-			(net "unconnected-(IC1-NC3-Pad8)")
-			(pinfunction "NC3_8")
-			(pintype "passive+no_connect")
+			(net "GND")
+			(pinfunction "GND_8")
+			(pintype "passive")
 		)
 		(pad "9" smd roundrect
@@
 			(layers "F.Cu" "F.Mask" "F.Paste")
 			(roundrect_rratio 0.25)
-			(net "unconnected-(IC1-NC4-Pad9)")
-			(pinfunction "NC4_9")
-			(pintype "passive+no_connect")
+			(net "GND")
+			(pinfunction "GND_9")
+			(pintype "passive")
 		)
 		(pad "10" smd roundrect
@@
 			(layers "F.Cu" "F.Mask" "F.Paste")
 			(roundrect_rratio 0.25)
-			(net "unconnected-(IC1-NC5-Pad10)")
-			(pinfunction "NC5_10")
-			(pintype "passive+no_connect")
+			(net "GND")
+			(pinfunction "GND_10")
+			(pintype "passive")
 		)
 		(pad "11" smd roundrect
@@
 			(layers "F.Cu" "F.Mask" "F.Paste")
 			(roundrect_rratio 0.25)
-			(net "unconnected-(IC1-NC6-Pad11)")
-			(pinfunction "NC6_11")
-			(pintype "passive+no_connect")
+			(net "GND")
+			(pinfunction "GND_11")
+			(pintype "passive")
 		)
 		(pad "12" smd roundrect
@@
 			(layers "F.Cu" "F.Mask" "F.Paste")
 			(roundrect_rratio 0.25)
-			(net "unconnected-(IC1-NC7-Pad12)")
-			(pinfunction "NC7_12")
-			(pintype "passive+no_connect")
+			(net "GND")
+			(pinfunction "GND_12")
+			(pintype "passive")
 		)
 		(pad "13" smd roundrect

Commit message: build(lib): use the kicad-common library
Own parts now come from the shared kicad-common submodule instead of
copies in external/. IC1 and the logo point to solar_cooker, with the
same netlist and ERC/DRC results.
Parts:
- G***: footprint external_footprints:logo -> solar_cooker:solar_cooker_logo
Changed lines of the file:
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@@
 		)
 	)
-	(footprint "external_footprints:logo"
+	(footprint "solar_cooker:solar_cooker_logo"
 		(layer "F.Cu")
 		(at 157 102.74)
